File: hardware/controller/components.kicad_sch (KiCad schematic)
At the start: 22 parts, among them SW1 EVP-ASAC1A, SW2 CL-SB-13A-02T, SW3 EVP-ASAC1A, SW4 EVP-ASAC1A, SW5 EVP-ASAC1A, SW6 EVP-ASAC1A

Commit message: renaming parts for consistency
Parts:
- C1, C4: JLCPCB Part # C15849 -> (none); LCSC Part # (none) -> C15849
- C2, C3: JLCPCB Part # C1525 -> (none); LCSC Part # (none) -> C1525
- CGQ1: JLCPCB # C91447 -> (none); LCSC Part # (none) -> C91447
- MK1: JLCPCB Part # C5656610 -> (none); LCSC Part # (none) -> C5656610
- R1, R10, R4, R5, R6, R7, R8, R9: JLCPCB Part # C25804 -> (none); LCSC Part # (none) -> C25804
- R2: JLCPCB Part # C25803 -> (none); LCSC Part # (none) -> C25803
- R3: JLCPCB Part # C22775 -> (none); LCSC Part # (none) -> C22775
- SW1, SW3, SW4, SW5, SW6: JLCPCB # C4365033 -> (none); LCSC Part # (none) -> C4365033
- SW2: LCSC Part C2921655 -> (none); LCSC Part # (none) -> C2921655
Changed lines of the file:
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@@
 			)
 		)
-		(property "LCSC Part Number" ""
-			(at 73.66 104.14 90)
-			(hide yes)
-			(show_name no)
-			(do_not_autoplace no)
-			(effects
-				(font
-					(size 1.27 1.27)
-				)
-			)
-		)
-		(property "JLCPCB Part #" "C22775"
+		(property "LCSC Part #" "C22775"
 			(at 73.66 104.14 0)
 			(hide yes)
@@
 			)
 		)
-		(property "JLCPCB Part #" "C1525"
+		(property "LCSC Part #" "C1525"
 			(at 34.925 47.625 0)
 			(hide yes)
@@
 			)
 		)
-		(property "JLCPCB Part #" "C15849"
+		(property "LCSC Part #" "C15849"
 			(at 73.66 115.57 0)
 			(hide yes)
@@
 			)
 		)
-		(property "LCSC Part" "C2921655"
+		(property "LCSC Part #" "C2921655"
 			(at 159.385 139.7 0)
 			(hide yes)
@@
 			)
 		)
-		(property "JLCPCB #" "C4365033"
+		(property "LCSC Part #" "C4365033"
 			(at 262.89 77.47 0)
 			(hide yes)
@@
 			)
 		)
-		(property "JLCPCB Part #" "C1525"
+		(property "LCSC Part #" "C1525"
 			(at 61.595 115.57 0)
 			(hide yes)
@@
 			)
 		)
-		(property "JLCPCB Part #" "C25804"
+		(property "LCSC Part #" "C25804"
 			(at 216.535 27.305 0)
 			(hide yes)
@@
 			)
 		)
-		(property "JLCPCB Part #" "C25804"
+		(property "LCSC Part #" "C25804"
 			(at 256.54 53.34 0)
 			(hide yes)
@@
 			)
 		)
-		(property "JLCPCB #" "C4365033"
+		(property "LCSC Part #" "C4365033"
 			(at 184.15 51.435 0)
 			(hide yes)
@@
 			)
 		)
-		(property "JLCPCB Part #" "C25804"
+		(property "LCSC Part #" "C25804"
 			(at 137.795 27.305 0)
 			(hide yes)
@@
 			)
 		)
-		(property "JLCPCB #" "C4365033"
+		(property "LCSC Part #" "C4365033"
 			(at 144.145 51.435 0)
 			(hide yes)
@@
 			)
 		)
-		(property "JLCPCB Part #" "C25804"
+		(property "LCSC Part #" "C25804"
 			(at 47.625 47.625 0)
 			(hide yes)
@@
 			)
 		)
-		(property "JLCPCB Part #" "C25804"
+		(property "LCSC Part #" "C25804"
 			(at 256.54 27.305 0)
 			(hide yes)
@@
 			)
 		)
-		(property "JLCPCB Part #" "C25804"
+		(property "LCSC Part #" "C25804"
 			(at 142.875 125.73 0)
 			(hide yes)
@@
 			)
 		)
-		(property "JLCPCB Part #" "C15849"
+		(property "LCSC Part #" "C15849"
 			(at 22.225 47.625 0)
 			(hide yes)
@@
 			)
 		)
-		(property "JLCPCB Part #" "C25804"
+		(property "LCSC Part #" "C25804"
 			(at 174.625 125.73 0)
 			(hide yes)
@@
 			)
 		)
-		(property "JLCPCB Part #" "C25803"
+		(property "LCSC Part #" "C25803"
 			(at 69.215 47.625 90)
 			(hide yes)
@@
 			)
 		)
-		(property "JLCPCB Part #" "C5656610"
+		(property "LCSC Part #" "C5656610"
 			(at 57.785 38.735 0)
 			(hide yes)
@@
 			)
 		)
-		(property "JLCPCB #" "C91447"
+		(property "LCSC Part #" "C91447"
 			(at 31.75 93.98 0)
 			(hide yes)
@@
 			)
 		)
-		(property "JLCPCB Part #" "C25804"
+		(property "LCSC Part #" "C25804"
 			(at 177.8 27.305 0)
 			(hide yes)
@@
 			)
 		)
-		(property "JLCPCB #" "C4365033"
+		(property "LCSC Part #" "C4365033"
 			(at 222.885 51.435 0)
 			(hide yes)
@@
 			)
 		)
-		(property "JLCPCB #" "C4365033"
+		(property "LCSC Part #" "C4365033"
 			(at 262.89 51.435 0)
 			(hide yes)

Commit message: adding some more stuff
Parts:
- added H1, H2, H3, H4: MountingHole, MountingHole:MountingHole_3.2mm_M3_Pad, symbol Mechanical:MountingHole

Commit message: controller layout work
Connections:
- net +3.3V: now also SW2.3; no longer R5.1, R6.1, SW2.1, SW2.4
- net GND: no longer SW2.3
- new net SOUND REACTIVE OFF: R6.1, SW2.4
- new net SOUND REACTIVE ON: R5.1, SW2.1
Other:
- moved on the sheet: R5, R6
