File: hardware/controller/components.kicad_sch (KiCad schematic)
At the start: 26 parts, among them SW1 EVP-ASAC1A, SW2 CL-SB-13A-02T, SW3 EVP-ASAC1A, SW4 EVP-ASAC1A, SW5 EVP-ASAC1A, SW6 EVP-ASAC1A

Commit message: feedback on the controller
Other:
- note added: "I think this is a 3-position switch, and I think you've made it so that in the middle position shorts 3.3V to GND?"
- note added: "Where did this 100-ohm resistor come from? Is that from a reference design? it seems rather high."
Changed lines of the file:
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@@
+		)
+	)
+	(text "I think this is a 3-position switch, and I think you've\nmade it so that in the middle position shorts 3.3V to GND?"
+		(exclude_from_sim no)
+		(at 148.844 143.256 0)
+		(effects
+			(font
+				(size 1.27 1.27)
+				(color 238 0 0 1)
+			)
+		)
+	)
+	(text "Where did this 100-ohm resistor come from?\nIs that from a reference design? it seems\nrather high."
+		(exclude_from_sim no)
+		(at 98.044 100.076 0)
+		(effects
+			(font
+				(size 1.27 1.27)
+				(color 238 0 0 1)
+			)
 		)
 	)

Commit message: fix up a few more things based on feedback
Parts:
- removed C4: 1µF, Capacitor_SMD:C_0603_1608Metric, symbol Device:C
- added C30: 4.7µF, Capacitor_SMD:C_0603_1608Metric, symbol Device:C
- added R11: (no value), Resistor_SMD:R_0603_1608Metric, symbol Device:R_US
Connections:
- net GND: now also C30.1, R11.2; no longer SW2.2
- net at C3.1, CGQ1.4 (VCC), R3.1: now also C30.2
- new net: R11.1, SW2.2
Other:
- note removed: "I think this is a 3-position switch, and I think you've made it so that in the middle position shorts 3.3V to GND?"
- note removed: "Where did this 100-ohm resistor come from? Is that from a reference design? it seems rather high."
Changed lines of the file:
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@@
-		)
-	)
-	(text "I think this is a 3-position switch, and I think you've\nmade it so that in the middle position shorts 3.3V to GND?"
-		(exclude_from_sim no)
-		(at 148.844 143.256 0)
-		(effects
-			(font
-				(size 1.27 1.27)
-				(color 238 0 0 1)
-			)
-		)
-	)
-	(text "Where did this 100-ohm resistor come from?\nIs that from a reference design? it seems\nrather high."
-		(exclude_from_sim no)
-		(at 98.044 100.076 0)
-		(effects
-			(font
-				(size 1.27 1.27)
-				(color 238 0 0 1)
-			)
 		)
 	)
@@
 	)
 	(junction
-		(at 73.66 111.76)
-		(diameter 0)
-		(color 0 0 0 0)
-	)
-	(junction
 		(at 142.875 126.365)
 		(diameter 0)
@@
 	)
 	(junction
+		(at 73.66 111.76)
+		(diameter 0)
+		(color 0 0 0 0)
+	)
+	(junction
 		(at 216.535 33.655)
 		(diameter 0)
@@
 	(wire
 		(pts
-			(xy 156.845 121.92) (xy 156.845 133.985)
+			(xy 156.845 121.92) (xy 156.845 125.73)
+		)
+		(stroke
+			(width 0)
+			(type default)
+		)
+	)
+	(wire
+		(pts
+			(xy 156.845 133.35) (xy 156.845 133.985)
 		)
 		(stroke
@@
 				(path "/ed43b915-8637-4fab-a1d1-340d9f2c05b8"
 					(reference "#PWR029")
+					(unit 1)
+				)
+			)
+		)
+	)
+	(symbol
+		(lib_id "Device:R_US")
+		(at 156.845 129.54 0)
+		(unit 1)
+		(body_style 1)
+		(exclude_from_sim no)
+		(in_bom yes)
+		(on_board yes)
+		(in_pos_files yes)
+		(dnp yes)
+		(property "Reference" "R11"
+			(at 152.4 130.81 0)
+			(show_name no)
+			(do_not_autoplace no)
+			(effects
+				(font
+					(size 1.27 1.27)
+				)
+			)
+		)
+		(property "Value" ""
+			(at 152.4 128.27 0)
+			(show_name no)
+			(do_not_autoplace no)
+			(effects
+				(font
+					(size 1.27 1.27)
+				)
+			)
+		)
+		(property "Footprint" "Resistor_SMD:R_0603_1608Metric"
+			(at 157.861 129.794 90)
+			(hide yes)
+			(show_name no)
+			(do_not_autoplace no)
+			(effects
+				(font
+					(size 1.27 1.27)
+				)
+			)
+		)
+		(property "Datasheet" ""
+			(at 156.845 129.54 0)
+			(hide yes)
+			(show_name no)
+			(do_not_autoplace no)
+			(effects
+				(font
+					(size 1.27 1.27)
+				)
+			)
+		)
+		(property "Description" "Resistor, US symbol"
+			(at 156.845 129.54 0)
+			(hide yes)
+			(show_name no)
+			(do_not_autoplace no)
+			(effects
+				(font
+					(size 1.27 1.27)
+				)
+			)
+		)
+		(property "LCSC Part #" ""
+			(at 156.845 129.54 0)
+			(hide yes)
+			(show_name no)
+			(do_not_autoplace no)
+			(effects
+				(font
+					(size 1.27 1.27)
+				)
+			)
+		)
+		(pin "1"
+		)
+		(pin "2"
+		)
+		(instances
+			(project "controller"
+				(path "/ed43b915-8637-4fab-a1d1-340d9f2c05b8"
+					(reference "R11")
 					(unit 1)
 				)
@@
 	)
 	(symbol
-		(lib_id "Device:C")
-		(at 73.66 115.57 0)
-		(unit 1)
-		(body_style 1)
-		(exclude_from_sim no)
-		(in_bom yes)
-		(on_board yes)
-		(in_pos_files yes)
-		(dnp no)
-		(property "Reference" "C4"
-			(at 80.01 114.3 0)
-			(show_name no)
-			(do_not_autoplace no)
-			(effects
-				(font
-					(size 1.27 1.27)
-				)
-			)
-		)
-		(property "Value" "1µF"
-			(at 80.01 116.84 0)
-			(show_name no)
-			(do_not_autoplace no)
-			(effects
-				(font
-					(size 1.27 1.27)
-				)
-			)
-		)
-		(property "Footprint" "Capacitor_SMD:C_0603_1608Metric"
-			(at 74.6252 119.38 0)
-			(hide yes)
-			(show_name no)
-			(do_not_autoplace no)
-			(effects
-				(font
-					(size 1.27 1.27)
-				)
-			)
-		)
-		(property "Datasheet" "https://jlcpcb.com/api/file/downloadByFileSystemAccessId/8556213788459761664"
-			(at 73.66 115.57 0)
-			(hide yes)
-			(show_name no)
-			(do_not_autoplace no)
-			(effects
-				(font
-					(size 1.27 1.27)
-				)
-			)
-		)
-		(property "Description" "Unpolarized capacitor"
-			(at 73.66 115.57 0)
-			(hide yes)
-			(show_name no)
-			(do_not_autoplace no)
-			(effects
-				(font
-					(size 1.27 1.27)
-				)
-			)
-		)
-		(property "LCSC Part #" "C15849"
-			(at 73.66 115.57 0)
-			(hide yes)
-			(show_name no)
-			(do_not_autoplace no)
-			(effects
-				(font
-					(size 1.27 1.27)
-				)
-			)
-		)
-		(pin "1"
-		)
-		(pin "2"
-		)
-		(instances
-			(project "controller"
-				(path "/ed43b915-8637-4fab-a1d1-340d9f2c05b8"
-					(reference "C4")
-					(unit 1)
-				)
-			)
-		)
-	)
-	(symbol
 		(lib_id "power:+3.3V")
 		(at 174.625 101.6 0)
@@
 					(unit 1)
 				)
+			)
+		)
+	)
+	(symbol
+		(lib_id "Device:C")
+		(at 73.66 115.57 180)
+		(unit 1)
+		(body_style 1)
+		(exclude_from_sim no)
+		(in_bom yes)
+		(on_board yes)
+		(in_pos_files yes)
+		(dnp no)
+		(fields_autoplaced yes)
+		(property "Reference" "C30"
+			(at 76.835 114.2999 0)
+			(show_name no)
+			(do_not_autoplace no)
+			(effects
+				(font
+					(size 1.27 1.27)
+				)
+				(justify right)
+			)
+		)
+		(property "Value" "4.7µF"
+			(at 76.835 116.8399 0)
+			(show_name no)
+			(do_not_autoplace no)
+			(effects
+				(font
+					(size 1.27 1.27)
+				)
+				(justify right)
+			)
+		)
+		(property "Footprint" "Capacitor_SMD:C_0603_1608Metric"
+			(at 72.6948 111.76 0)
+			(hide yes)
+			(show_name no)
+			(do_not_autoplace no)
+			(effects
+				(font
+					(size 1.27 1.27)
+				)
+			)
+		)
+		(property "Datasheet" "https://jlcpcb.com/api/file/downloadByFileSystemAccessId/8579707103462166528"
+			(at 73.66 115.57 0)
+			(hide yes)
+			(show_name no)
+			(do_not_autoplace no)
+			(effects
+				(font
+					(size 1.27 1.27)
+				)
+			)
+		)
+		(property "Description" "Unpolarized capacitor"
+			(at 73.66 115.57 0)
+			(hide yes)
+			(show_name no)
+			(do_not_autoplace no)
+			(effects
+				(font
+					(size 1.27 1.27)
+				)
+			)
+		)
+		(property "JLCPCB Part #" "C19666"
+			(at 73.66 115.57 90)
+			(hide yes)
+			(show_name no)
+			(do_not_autoplace no)
+			(effects
+				(font
+					(size 1.27 1.27)
+				)
+			)
+		)
+		(pin "1"
+		)
+		(pin "2"
+		)
+		(instances
+			(project "controller"
+				(path "/ed43b915-8637-4fab-a1d1-340d9f2c05b8"
+					(reference "C30")
+					(unit 1)
+				)

Commit message: tiny board update for controller
Parts:
- C30: JLCPCB Part # C19666 -> (none); LCSC Part # (none) -> C19666
- R11: now left out of the parts list
Changed lines of the file:
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@@
 		(body_style 1)
 		(exclude_from_sim no)
-		(in_bom yes)
+		(in_bom no)
 		(on_board yes)
 		(in_pos_files yes)
@@
 			)
 		)
-		(property "JLCPCB Part #" "C19666"
-			(at 73.66 115.57 90)
-			(hide yes)
-			(show_name no)
+		(property "LCSC Part #" "C19666"
+			(at 73.66 115.57 0)
+			(hide yes)
+			(show_name no)

Commit message: change a part on controller board, make production files
Parts:
- R1, R10, R4, R5, R6, R7, R8, R9: LCSC Part # C25804 -> C98220
