File: hardware/controller/voltage_converters.kicad_sch (KiCad schematic)
At the start: 26 parts, among them U10 XDJK-0051-025, U7 EA8212HT6R, U8 EA8212HT6R, U9 EA8212HT6R

Commit message: feedback on the controller
Parts:
- removed C11, C12, C17: 100nF, Capacitor_SMD:C_0402_1005Metric, symbol Device:C
- removed C13, C15, C19, C20: 10µF, Capacitor_SMD:C_0603_1608Metric, symbol Device:C
- removed C18: 47µF, Capacitor_SMD:C_1210_3225Metric, symbol Device:C
- removed L1, L3: MGFL2012F2R2MT-LF, easyeda2kicad:L0805, symbol easyeda2kicad:MGFL2012F2R2MT-LF
- removed R15, R19, R21, R23: 100kΩ, Resistor_SMD:R_0402_1005Metric, symbol Device:R_US
- removed R17: 732kΩ, Resistor_SMD:R_0402_1005Metric, symbol Device:R_US
- removed R22: 453kΩ, Resistor_SMD:R_0402_1005Metric, symbol Device:R_US
- removed U7, U9: EA8212HT6R, easyeda2kicad:SOT-23-6_L2.9-W1.6-P0.95-LS2.8-BR, symbol new:EA8212HT6R
- added C23, C24, C35: 10µF, Capacitor_SMD:C_0603_1608Metric, symbol Device:C
- added C27, C36: 33nF, Capacitor_SMD:C_0402_1005Metric, symbol Device:C
- L2: value MGFL2012F2R2MT-LF -> 4.7uH; footprint easyeda2kicad:L0805 -> Inductor_SMD:L_Changjiang_FNR4030S; LCSC Part # C281115 -> C167874; MPN MGFL2012F2R2MT-LF -> FNR4030S4R7MT; Manufacturer microgate(麦捷科技) -> changjiang
Connections:
- net +12V: now also C24.1, C35.1
- net +4V: now also C23.1, C36.2
- net GND: now also C23.2, C24.2, C35.2
- net at U8.1 (BOOT): now also C27.1
- net at L2.1, U8.6 (SWITCH): now also C27.2
- net at R16.1, R18.1, U8.3 (FBK): now also C36.1
Other:
- note added: "The Dabao can work off of 4 volts, so we don't need a separate 5V regulator"
- note added: "There's a 3.3V regulator on dabao that you can use"
- note removed: "VOLTAGE CONVERTER 12V -> 3.3V"
- note removed: "VOLTAGE CONVERTER 12V -> 5V"

Commit message: updates to schematic based on feedback
Parts:
- removed C36: 33nF, Capacitor_SMD:C_0402_1005Metric, symbol Device:C
Changed lines of the file:
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@@
-	)
-	(junction
-		(at 41.91 151.765)
-		(diameter 0)
-		(color 0 0 0 0)
 	)
 	(junction
@@
 	(wire
 		(pts
-			(xy 41.91 124.46) (xy 41.91 151.765)
-		)
-		(stroke
-			(width 0)
-			(type default)
-		)
-	)
-	(wire
-		(pts
 			(xy 211.455 129.54) (xy 221.615 129.54)
 		)
@@
 	(wire
 		(pts
-			(xy 41.91 151.765) (xy 41.91 158.115)
+			(xy 41.91 124.46) (xy 41.91 158.115)
 		)
 		(stroke
@@
 		(pts
 			(xy 221.615 129.54) (xy 221.615 124.46)
-		)
-		(stroke
-			(width 0)
-			(type default)
-		)
-	)
-	(wire
-		(pts
-			(xy 34.925 151.765) (xy 41.91 151.765)
 		)
 		(stroke
@@
 					(unit 1)
 				)
-			)
-		)
-	)
-	(symbol
-		(lib_id "Device:C")
-		(at 34.925 155.575 180)
-		(unit 1)
-		(body_style 1)
-		(exclude_from_sim no)
-		(in_bom yes)
-		(on_board yes)
-		(in_pos_files yes)
-		(dnp yes)
-		(property "Reference" "C36"
-			(at 29.845 156.845 0)
-			(show_name no)
-			(do_not_autoplace no)
-			(effects
-				(font
-					(size 1.27 1.27)
-				)
-				(justify left)
-			)
-		)
-		(property "Value" "33nF"
-			(at 31.115 154.94 0)
-			(show_name no)
-			(do_not_autoplace no)
-			(effects
-				(font
-					(size 1.27 1.27)
-				)
-				(justify left)
-			)
-		)
-		(property "Footprint" "Capacitor_SMD:C_0402_1005Metric"
-			(at 33.9598 151.765 0)
-			(hide yes)
-			(show_name no)
-			(do_not_autoplace no)
-			(effects
-				(font
-					(size 1.27 1.27)
-				)
-			)
-		)
-		(property "Datasheet" "https://www.lcsc.com/datasheet/lcsc_datasheet_2304140030_Samsung-Electro-Mechanics-CL05B104KO5NNNC_C1525.pdf"
-			(at 34.925 155.575 0)
-			(hide yes)
-			(show_name no)
-			(do_not_autoplace no)
-			(effects
-				(font
-					(size 1.27 1.27)
-				)
-			)
-		)
-		(property "Description" "Unpolarized capacitor"
-			(at 34.925 155.575 0)
-			(hide yes)
-			(show_name no)
-			(do_not_autoplace no)
-			(effects
-				(font
-					(size 1.27 1.27)
-				)
-			)
-		)
-		(property "LCSC Part #" "C507072"
-			(at 34.925 155.575 0)
-			(hide yes)
-			(show_name no)
-			(do_not_autoplace no)
-			(effects
-				(font
-					(size 1.27 1.27)
-				)
-			)
-		)
-		(pin "2"
-		)
-		(pin "1"
-		)
-		(instances
-			(project "controller"
-				(path "/95e5c331-6890-437f-94b9-bde400751ae8"
-					(reference "C36")
-					(unit 1)
-				)

Commit message: fix up a few more things based on feedback
Other:
- note removed: "The Dabao can work off of 4 volts, so we don't need a separate 5V regulator"
- note removed: "There's a 3.3V regulator on dabao that you can use"
- moved on the sheet: C14, C16, C23, C24, C27, C35, L2, R16, R18, R20, U10, U8
