File: hardware/controller/usb-c_to_triangles.kicad_sch (KiCad schematic)
At the start: 14 parts, among them J1 TYPE-C 16PLT-H10.0, J2 TYPE-C 16PLT-H10.0, U5 SN74LVC1T45DBV, U6 SN74LVC1T45DBV

Commit message: feedback on the controller
Parts:
- removed C10, C7: 47µF, Capacitor_SMD:C_1210_3225Metric, symbol Device:C
- removed R11, R12, R13, R14: 5.1kΩ, Resistor_SMD:R_0603_1608Metric, symbol Device:R_US
- added C33, C34: 10µF, Capacitor_SMD:C_0603_1608Metric, symbol Device:C
Connections:
- net +12V: now also C33.1, C34.1
- net GND: now also C33.2, C34.2

Commit message: board placement
Parts:
- removed C34: 10µF, Capacitor_SMD:C_0603_1608Metric, symbol Device:C
- added C3: 10µF, Capacitor_SMD:C_0603_1608Metric, symbol Device:C
- J1, J2: value TYPE-C 16PLT-H10.0 -> TYPE-C-31-M-12; footprint easyeda2kicad:TYPE-C-SMD_USB4120-03-C -> easyeda2kicad:USB-C_SMD-TYPE-C-31-M-12_1; symbol easyeda2kicad:TYPE-C16PLT-H10.0 -> easyeda2kicad:TYPE-C-31-M-12; LCSC Part # C3151749 -> C165948
- renumbered C5 to C1, C6 to C2, C8 to C4, C33 to C5, C9 to C6
Connections:
- net +12V: now also J1.A4B9 (VBUS), J1.B4A9 (VBUS), J2.A4B9 (VBUS), J2.B4A9 (VBUS), C3.1; no longer J1.A4 (VBUS), J1.A9 (VBUS), J1.B4 (VBUS), J1.B9 (VBUS), J2.A4 (VBUS), J2.A9 (VBUS), J2.B4 (VBUS), J2.B9 (VBUS)
- net GND: now also J1.1 (EH), J1.2 (EH), J1.3 (EH), J1.4 (EH), J1.A1B12 (GND), J1.B1A12 (GND), J2.1 (EH), J2.2 (EH), J2.3 (EH), J2.4 (EH), J2.A1B12 (GND), J2.B1A12 (GND), C3.2; no longer J1.0 (EH), J1.A1 (GND), J1.A12 (GND), J1.B1 (GND), J1.B12 (GND), J2.0 (EH), J2.A1 (GND), J2.A12 (GND), J2.B1 (GND), J2.B12 (GND)
- no-connect marks 4 -> 8
Other:
- moved on the sheet: C5
