File: hardware/controller/ear.kicad_sch (KiCad schematic)
At the start: 0 parts

Commit message: more schematic work
Parts:
- added C29, C31, C33, C37, C38: 100nF, Capacitor_SMD:C_0201_0603Metric, symbol Device:C
- added C32, C36, C41: 2.2µF, Capacitor_SMD:C_0201_0603Metric, symbol Device:C
- added C34, C40: 1µF, Capacitor_SMD:C_0201_0603Metric, symbol Device:C
- added C39, C42: 33pF, Capacitor_SMD:C_0201_0603Metric, symbol Device:C
- added D8, D9: ESD8351XV2T1G, easyeda2kicad:SOD-523_L1.2-W0.8-LS1.6-RD, symbol easyeda2kicad:ESD8351XV2T1G_C19829478
- added R26: 10kΩ, Resistor_SMD:R_0201_0603Metric, symbol Device:R_US
- added R28: 4.7MΩ, Resistor_SMD:R_0402_1005Metric, symbol Device:R_US
- added R30: 10kΩ, Resistor_SMD:R_0402_1005Metric, symbol Device:R_US
- added R31, R32: 5.1kΩ, Resistor_SMD:R_0402_1005Metric, symbol Device:R_US
- added TP3, TP4: TestPoint, TestPoint:TestPoint_Pad_D1.0mm, symbol Connector:TestPoint
- added U6: EMS4000RSW, easyeda2kicad:UQFN-10_L1.8-W1.4-P0.40-TL, symbol easyeda2kicad:EMS4000RSW
- added U7: baochip1x, baochip:WLCSP-71_9x8_4.062x3.762mm, symbol baochip:baochip1x
- added USBC4: TYPE-C-31-M-12, easyeda2kicad:USB-C_SMD-TYPE-C-31-M-12_1, symbol easyeda2kicad:TYPE-C-31-M-12
- added Y2: 48 MHz, Crystal:Crystal_SMD_3225-4Pin_3.2x2.5mm, symbol Device:Crystal_GND24
Connections:
- new net: C32.1, U7.C1 (VDD2.5)
- new net: TP3.1, U6.10 (SEL), U7.D1 (PC13)
- new net: C39.1, R28.1, U7.H1 (X48MI), Y2.1
- new net: C42.1, R28.2, U7.H2 (X48MO), Y2.3
- new net: U6.7 (L1+), U7.A2 (USB_D+)
- new net: U6.6 (L1-), U7.B1 (USB_D-)
- new net: C38.1, R26.2, U7.H5 (AORSTn)
- new net: R30.2, USBC4.A4B9 (VBUS), USBC4.B4A9 (VBUS)
- new net: R31.2, USBC4.A5 (CC1)
- new net: R32.2, USBC4.B5 (CC2)
- new net +0.85V: C37.1, C40.1, C41.1, U7.A4 (VDD.85), U7.E6 (VDDAO), U7.E7 (VDD.85), U7.F6 (PA6), U7.F7 (VDD.85)
- new net +3.3V: C29.1, C31.1, C33.1, C34.1, C36.1, R26.1, U6.9 (VDD), U7.A3 (V3.3IN), U7.B7 (VDDIO), U7.C6 (PF9_PA0), U7.C7 (VDDIO), U7.D6 (PB0), U7.D7 (PA7), U7.H4 (V3.3RR)
- new net AUDIO_LINK: U7.E9 (PB14)
- new net EAR_DATA_D+: D8.1 (C), U6.1 (C0+), USBC4.A6 (DP1), USBC4.B6 (DP2)
- new net EAR_DATA_D-: D9.1 (C), U6.2 (C0-), USBC4.A7 (DN1), USBC4.B7 (DN2)
- new net GND: C29.2, C31.2, C32.2, C33.2, C34.2, C36.2, C37.2, C38.2, C39.2, C40.2, C41.2, C42.2, D8.2 (A), D9.2 (A), R30.1, R31.1, R32.1, TP4.1, U6.3 (GND), U6.4 (L0-), U6.5 (L0+), U6.8 (~{EN}), U7.B2 (GND), U7.C3 (GND), U7.C4 (PA5), U7.C5 (GND), U7.D4 (GND), U7.D5 (GND_TP), U7.E3 (PC5), U7.E4 (PF1), U7.F3 (PA3), U7.F4 (PC6), U7.F5 (GND), USBC4.1 (EH), USBC4.2 (EH), USBC4.3 (EH), USBC4.4 (EH), USBC4.A1B12 (GND), USBC4.B1A12 (GND), Y2.2 (G), Y2.4 (G)
- no-connect marks 0 -> 8

Commit message: first round of schematic v3 done
Connections:
- net MIC WS: now reaches U7.A7 (PB3)
- net MIC DATA OUTPUT: now reaches U7.A8 (PB2)
- net MIC CLOCK: now reaches U7.A9 (PB1)
- no-connect marks 8 -> 39
Other:
- moved on the sheet: C29, C31, C32, C33, C34, C36, C37, C38, C40, C41, C42, D8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

Commit message: adding power flags so the schematic passes erc
Changed lines of the file:
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@@
 	(paper "A4")
 	(junction
+		(at 31.75 175.26)
+		(diameter 0)
+		(color 0 0 0 0)
+	)
+	(junction
 		(at 66.04 175.26)
 		(diameter 0)
@@
 					(unit 1)
 				)
+			)
+		)
+	)
+	(symbol
+		(lib_id "power:PWR_FLAG")
+		(at 31.75 175.26 0)
+		(unit 1)
+		(body_style 1)
+		(exclude_from_sim no)
+		(in_bom yes)
+		(on_board yes)
+		(in_pos_files yes)
+		(dnp no)
+		(fields_autoplaced yes)
+		(property "Reference" "#FLG06"
+			(at 31.75 173.355 0)
+			(hide yes)
+			(show_name no)
+			(do_not_autoplace no)
+			(effects
+				(font
+					(size 1.27 1.27)
+				)
+			)
+		)
+		(property "Value" "PWR_FLAG"
+			(at 30.48 171.45 0)
+			(show_name no)
+			(do_not_autoplace no)
+			(effects
+				(font
+					(size 1.27 1.27)
+				)
+			)
+		)
+		(property "Footprint" ""
+			(at 31.75 175.26 0)
+			(hide yes)
+			(show_name no)
+			(do_not_autoplace no)
+			(effects
+				(font
+					(size 1.27 1.27)
+				)
+			)
+		)
+		(property "Datasheet" ""
+			(at 31.75 175.26 0)
+			(hide yes)
+			(show_name no)
+			(do_not_autoplace no)
+			(effects
+				(font
+					(size 1.27 1.27)
+				)
+			)
+		)
+		(property "Description" "Special symbol for telling ERC where power comes from"
+			(at 31.75 175.26 0)
+			(hide yes)
+			(show_name no)
+			(do_not_autoplace no)
+			(effects
+				(font
+					(size 1.27 1.27)
+				)
+			)
+		)
+		(pin "1"
+		)
+		(instances
+			(project "controller"
+				(path "/dab966ac-748d-4912-886d-b156bece3c93/3bb67c02-3594-463f-8de9-69338cd90bb8"
+					(reference "#FLG06")
+					(unit 1)
+				)
