File: hardware/controller/ear.kicad_sch (KiCad schematic)
At the start: 25 parts, among them U6 EMS4000RSW, U7 baochip1x, Y2 48 MHz

Commit message: tidying up schematic and drawing outline for board
Parts:
- renumbered C29 to C23, C31 to C24, C32 to C25, C33 to C26, C34 to C27, C36 to C28, C37 to C29, C38 to C30, C39 to C31, C40 to C32, C41 to C33, C42 to C34, R26 to R13, R28 to R14, R30 to R15, R31 to R16, R32 to R17

Commit message: welcome to the pcb, parts
Parts:
- TP3, TP4: now left out of the parts list
Changed lines of the file:
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@@
 		(body_style 1)
 		(exclude_from_sim no)
-		(in_bom yes)
-		(on_board yes)
-		(in_pos_files yes)
+		(in_bom no)
+		(on_board yes)
+		(in_pos_files no)
 		(dnp no)
 		(fields_autoplaced yes)
@@
 		(body_style 1)
 		(exclude_from_sim no)
-		(in_bom yes)
-		(on_board yes)
-		(in_pos_files yes)
-		(dnp no)
-		(fields_autoplaced yes)
+		(in_bom no)
+		(on_board yes)
+		(in_pos_files no)
+		(dnp no)
+		(fields_autoplaced yes)
