File: hardware/controller/power_and_tiles.kicad_sch (KiCad schematic)
At the start: 27 parts, among them U1 XDJK-0051-025, U2 EA8212HT6R, U3 MT3406

Commit message: hooking up parts in the schematic
Parts:
- removed C4: 33nF, Capacitor_SMD:C_0402_1005Metric, symbol Device:C
- removed C5, C6: 10µF, Capacitor_SMD:C_0603_1608Metric, symbol Device:C
- removed L1: 4.7µH, Inductor_SMD:L_Changjiang_FNR4030S, symbol Device:L
- removed R10, R11: 100kΩ, Resistor_SMD:R_0402_1005Metric, symbol Device:R_US
- removed R13: 10kΩ, Resistor_SMD:R_0402_1005Metric, symbol Device:R_US
- removed U1: XDJK-0051-025, easyeda2kicad:DC-IN-TH_XDJK-0051-025, symbol easyeda2kicad:XDJK-0051-025
- removed U2: EA8212HT6R, easyeda2kicad:SOT-23-6_L2.9-W1.6-P0.95-LS2.8-BR, symbol easyeda2kicad:EA8212HT6R
- added C24, C26, C35: 10µF, Capacitor_SMD:C_0603_1608Metric, symbol Device:C
- added C27: 33nF, Capacitor_SMD:C_0402_1005Metric, symbol Device:C
- added L3: 4.7µH, Inductor_SMD:L_Changjiang_FNR4030S, symbol Device:L
- added R27, R29: 100kΩ, Resistor_SMD:R_0402_1005Metric, symbol Device:R_US
- added U10: XDJK-0051-025, easyeda2kicad:DC-IN-TH_XDJK-0051-025, symbol easyeda2kicad:XDJK-0051-025
- added U8: EA8212HT6R, easyeda2kicad:SOT-23-6_L2.9-W1.6-P0.95-LS2.8-BR, symbol easyeda2kicad:EA8212HT6R
Connections:
- net +3.3V: now reaches C10.1
- net +3.3V: now also C7.1, C9.1, R9.2, U3.1 (EN), U3.4 (VIN), L3.2
- net GND: now reaches C10.2
- net GND: now also C7.2, C8.2, C9.2, D1.2 (A), R16.2, U3.2 (GND), C24.2, C26.2, C35.2, R27.2, U10.2, U8.2 (GND)
- net +0.85V: now reaches L2.1
- net +0.85V: now also C8.1, R12.1
- net at L2.2: now also U3.3 (SW)
- net at R16.1: now also R12.2, U3.5 (FB)
- net at R9.1: now also R27.1, U8.3 (FBK)
- net +12V: now reaches D1.1 (K)
- net +12V: now also C24.1, C26.1, C35.1, R29.2, U10.1, U8.5 (PWR)
- new net: C27.1, U8.1 (BOOT)
- new net: C27.2, L3.1, U8.6 (SWITCH)
- new net: R29.1, U8.4 (RUN)
- no-connect marks 0 -> 1
Other:
- note added: "12V POWER BARREL CONNECTOR"
- note added: "VOLTAGE CONVERTER 12V -> 3.3V"
- note added: "VOLTAGE CONVERTER 3.3V -> 0.85V"
- moved on the sheet: C10, C7, C8, C9, D1, L2, R12, R16, R9, U3

Commit message: power and tiles schematic work
Parts:
- added C25, C28: 10µF, Capacitor_SMD:C_0603_1608Metric, symbol Device:C
Connections:
- net +12V: now also D2.1 (K), D3.1 (K), USBC1.A4B9 (VBUS), USBC1.B4A9 (VBUS), USBC2.A4B9 (VBUS), USBC2.B4A9 (VBUS), C25.1, C28.1
- net GND: now also D2.2 (A), D3.2 (A), D4.2 (A), D5.2 (A), USBC1.1 (EH), USBC1.2 (EH), USBC1.3 (EH), USBC1.4 (EH), USBC1.A1B12 (GND), USBC1.B1A12 (GND), USBC2.1 (EH), USBC2.2 (EH), USBC2.3 (EH), USBC2.4 (EH), USBC2.A1B12 (GND), USBC2.B1A12 (GND), C25.2, C28.2
- net at USBC1.A6 (DP1): now also D4.1 (C), R14.2, USBC1.A7 (DN1), USBC1.B6 (DP2), USBC1.B7 (DN2)
- net at D5.1 (C): now also R15.2, USBC2.A6 (DP1), USBC2.A7 (DN1), USBC2.B6 (DP2), USBC2.B7 (DN2)
- net LED_DATA_1: now reaches R14.1
- net LED_DATA_2: now reaches R15.1
- no-connect marks 1 -> 9
Other:
- note added: "USB TO TRIANGLES 1-12"
- note added: "USB TO TRIANGLES 13-25"
- moved on the sheet: C10, C24, C26, C27, C9, D2, D4, L3, R14, R27, R29, R9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

Commit message: tidying up schematic and drawing outline for board
Parts:
- renumbered C8 to C1, C28 to C10, C27 to C2, C7 to C3, C24 to C4, C9 to C5, C26 to C6, C10 to C7, C35 to C8, C25 to C9, D4 to D1, D1 to D2, D2 to D3, D5 to D4, D3 to D5, L2 to L1, L3 to L2, R27 to R1, R9 to R2, R12 to R3, R16 to R4, R29 to R5, R14 to R6, R15 to R7, U8 to U1, U3 to U2, U10 to U3
