File: hardware/triangle/triangle.kicad_pcb (KiCad board)
At the start: 4 copper layers, 100 x 86.6 mm, 72 parts, among them J1 USB_C_Receptacle_USB2.0_16P, J2 USB_C_Receptacle_USB2.0_16P, U2 EA8212HT6R

Commit message: triangel review
Parts:
- removed C25, C29: 47µF, Capacitor_SMD:C_1206_3216Metric
- removed R5, R6, R7, R8: 5.1kΩ, Resistor_SMD:R_0603_1608Metric
- added C30: 10µF, Capacitor_SMD:C_0603_1608Metric, B.Cu at (134.1, 135.3)
- added C31: 10µF, Capacitor_SMD:C_0603_1608Metric, B.Cu at (174.2, 122.0)
- added C32: 33nF, Capacitor_SMD:C_0402_1005Metric, B.Cu at (175.1, 126.4)
- added C33: 10µF, Capacitor_SMD:C_0603_1608Metric, B.Cu at (145.3, 104.7)
- added C34: 10µF, Capacitor_SMD:C_0603_1608Metric, B.Cu at (172.7, 131.1)
- C26: value 100nF -> 33nF
- L1: value MGFL2012F2R2MT-LF -> 4.7uH; footprint footprints:L0805 -> Inductor_SMD:L_Changjiang_FNR4030S
- TP1-4V1: renamed from TP1 4V
- TP2-LED_DATA_IN1: renamed from TP2 DATA_IN
- TP3-LED_DATA_OUT1: renamed from TP3 DATA_OUT
- moved C28 4.55 mm to (172.7, 122.9)
- moved C27 4.49 mm to (171.9, 129.8), turned to 30 degrees
- moved L1 1.46 mm to (169.0, 120.5), turned to 30 degrees
- moved R3 0.59 mm to (175.5, 127.7)
Connections:
- J1 pad A5: Net-(J1-CC1) -> unconnected-(J1-CC1-PadA5)
- J1 pad B5: Net-(J1-CC2) -> unconnected-(J1-CC2-PadB5)
- J2 pad A5: Net-(J2-CC1) -> unconnected-(J2-CC1-PadA5)
- J2 pad B5: Net-(J2-CC2) -> unconnected-(J2-CC2-PadB5)
Routing:
- net +12V: track 28.5 -> 16.0 mm, vias 5 -> 0
- net GND: track 108.0 -> 101.5 mm, vias 28 -> 30
- net Net-(J1-CC2): track 5.33 -> 0.00 mm
- net Net-(J1-CC1): track 3.81 -> 0.00 mm
- net Net-(J2-CC1): track 3.31 -> 0.00 mm
- net Net-(J2-CC2): track 3.13 -> 0.00 mm
- net +4V: track 109.8 -> 112.4 mm, vias 27 -> 28
- net Net-(U2-SWITCH): track 4.27 -> 5.16 mm
- net Net-(U2-FBK): track 3.44 -> 4.06 mm
- added copper zone on B.Cu, net +12V
