File: hardware/triangle/triangle.kicad_sch (KiCad schematic)
At the start: 56 parts

Commit message: rearranging shared files and input board beginnings
Parts:
- D1, D10, D11, D12, D13, D14, D15, D16, D17, D18, D19, D2, D20, D21, D22, D23, D24, D3, D4, D5, D6, D7, D8, D9: footprint footprints:LED_WS2812B-2020_PLCC4_2.0x2.0mm - no silkscreen -> easyeda2kicad:LED_WS2812B-2020_PLCC4_2.0x2.0mm - no silkscreen
Changed lines of the file:
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@@
 			)
 		)
-		(property "Footprint" "footprints:LED_WS2812B-2020_PLCC4_2.0x2.0mm - no silkscreen"
+		(property "Footprint" "easyeda2kicad:LED_WS2812B-2020_PLCC4_2.0x2.0mm - no silkscreen"
 			(at 146.685 43.18 0)
 			(hide yes)
@@
 			)
 		)
-		(property "Footprint" "footprints:LED_WS2812B-2020_PLCC4_2.0x2.0mm - no silkscreen"
+		(property "Footprint" "easyeda2kicad:LED_WS2812B-2020_PLCC4_2.0x2.0mm - no silkscreen"
 			(at 206.375 51.435 0)
 			(hide yes)
@@
 			)
 		)
-		(property "Footprint" "footprints:LED_WS2812B-2020_PLCC4_2.0x2.0mm - no silkscreen"
+		(property "Footprint" "easyeda2kicad:LED_WS2812B-2020_PLCC4_2.0x2.0mm - no silkscreen"
 			(at 102.87 43.18 0)
 			(hide yes)
@@
 			)
 		)
-		(property "Footprint" "footprints:LED_WS2812B-2020_PLCC4_2.0x2.0mm - no silkscreen"
+		(property "Footprint" "easyeda2kicad:LED_WS2812B-2020_PLCC4_2.0x2.0mm - no silkscreen"
 			(at 124.46 43.18 0)
 			(hide yes)
@@
 			)
 		)
-		(property "Footprint" "footprints:LED_WS2812B-2020_PLCC4_2.0x2.0mm - no silkscreen"
+		(property "Footprint" "easyeda2kicad:LED_WS2812B-2020_PLCC4_2.0x2.0mm - no silkscreen"
 			(at 252.73 43.18 0)
 			(hide yes)
@@
 			)
 		)
-		(property "Footprint" "footprints:LED_WS2812B-2020_PLCC4_2.0x2.0mm - no silkscreen"
+		(property "Footprint" "easyeda2kicad:LED_WS2812B-2020_PLCC4_2.0x2.0mm - no silkscreen"
 			(at 102.87 96.52 0)
 			(hide yes)
@@
 			)
 		)
-		(property "Footprint" "footprints:LED_WS2812B-2020_PLCC4_2.0x2.0mm - no silkscreen"
+		(property "Footprint" "easyeda2kicad:LED_WS2812B-2020_PLCC4_2.0x2.0mm - no silkscreen"
 			(at 124.46 96.52 0)
 			(hide yes)
@@
 			)
 		)
-		(property "Footprint" "footprints:LED_WS2812B-2020_PLCC4_2.0x2.0mm - no silkscreen"
+		(property "Footprint" "easyeda2kicad:LED_WS2812B-2020_PLCC4_2.0x2.0mm - no silkscreen"
 			(at 121.92 51.435 0)
 			(hide yes)
@@
 			)
 		)
-		(property "Footprint" "footprints:LED_WS2812B-2020_PLCC4_2.0x2.0mm - no silkscreen"
+		(property "Footprint" "easyeda2kicad:LED_WS2812B-2020_PLCC4_2.0x2.0mm - no silkscreen"
 			(at 250.19 51.435 0)
 			(hide yes)
@@
 			)
 		)
-		(property "Footprint" "footprints:LED_WS2812B-2020_PLCC4_2.0x2.0mm - no silkscreen"
+		(property "Footprint" "easyeda2kicad:LED_WS2812B-2020_PLCC4_2.0x2.0mm - no silkscreen"
 			(at 146.685 96.52 0)
 			(hide yes)
@@
 			)
 		)
-		(property "Footprint" "footprints:LED_WS2812B-2020_PLCC4_2.0x2.0mm - no silkscreen"
+		(property "Footprint" "easyeda2kicad:LED_WS2812B-2020_PLCC4_2.0x2.0mm - no silkscreen"
 			(at 184.785 51.435 0)
 			(hide yes)
@@
 			)
 		)
-		(property "Footprint" "footprints:LED_WS2812B-2020_PLCC4_2.0x2.0mm - no silkscreen"
+		(property "Footprint" "easyeda2kicad:LED_WS2812B-2020_PLCC4_2.0x2.0mm - no silkscreen"
 			(at 252.73 96.52 0)
 			(hide yes)
@@
 			)
 		)
-		(property "Footprint" "footprints:LED_WS2812B-2020_PLCC4_2.0x2.0mm - no silkscreen"
+		(property "Footprint" "easyeda2kicad:LED_WS2812B-2020_PLCC4_2.0x2.0mm - no silkscreen"
 			(at 168.275 43.18 0)
 			(hide yes)
@@
 			)
 		)
-		(property "Footprint" "footprints:LED_WS2812B-2020_PLCC4_2.0x2.0mm - no silkscreen"
+		(property "Footprint" "easyeda2kicad:LED_WS2812B-2020_PLCC4_2.0x2.0mm - no silkscreen"
 			(at 228.6 51.435 0)
 			(hide yes)
@@
 			)
 		)
-		(property "Footprint" "footprints:LED_WS2812B-2020_PLCC4_2.0x2.0mm - no silkscreen"
+		(property "Footprint" "easyeda2kicad:LED_WS2812B-2020_PLCC4_2.0x2.0mm - no silkscreen"
 			(at 210.185 43.18 0)
 			(hide yes)
@@
 			)
 		)
-		(property "Footprint" "footprints:LED_WS2812B-2020_PLCC4_2.0x2.0mm - no silkscreen"
+		(property "Footprint" "easyeda2kicad:LED_WS2812B-2020_PLCC4_2.0x2.0mm - no silkscreen"
 			(at 231.14 43.18 0)
 			(hide yes)
@@
 			)
 		)
-		(property "Footprint" "footprints:LED_WS2812B-2020_PLCC4_2.0x2.0mm - no silkscreen"
+		(property "Footprint" "easyeda2kicad:LED_WS2812B-2020_PLCC4_2.0x2.0mm - no silkscreen"
 			(at 189.865 43.18 0)
 			(hide yes)
@@
 			)
 		)
-		(property "Footprint" "footprints:LED_WS2812B-2020_PLCC4_2.0x2.0mm - no silkscreen"
+		(property "Footprint" "easyeda2kicad:LED_WS2812B-2020_PLCC4_2.0x2.0mm - no silkscreen"
 			(at 142.875 51.435 0)
 			(hide yes)
@@
 			)
 		)
-		(property "Footprint" "footprints:LED_WS2812B-2020_PLCC4_2.0x2.0mm - no silkscreen"
+		(property "Footprint" "easyeda2kicad:LED_WS2812B-2020_PLCC4_2.0x2.0mm - no silkscreen"
 			(at 163.195 51.435 0)
 			(hide yes)
@@
 			)
 		)
-		(property "Footprint" "footprints:LED_WS2812B-2020_PLCC4_2.0x2.0mm - no silkscreen"
+		(property "Footprint" "easyeda2kicad:LED_WS2812B-2020_PLCC4_2.0x2.0mm - no silkscreen"
 			(at 189.865 96.52 0)
 			(hide yes)
@@
 			)
 		)
-		(property "Footprint" "footprints:LED_WS2812B-2020_PLCC4_2.0x2.0mm - no silkscreen"
+		(property "Footprint" "easyeda2kicad:LED_WS2812B-2020_PLCC4_2.0x2.0mm - no silkscreen"
 			(at 100.33 51.435 0)
 			(hide yes)
@@
 			)
 		)
-		(property "Footprint" "footprints:LED_WS2812B-2020_PLCC4_2.0x2.0mm - no silkscreen"
+		(property "Footprint" "easyeda2kicad:LED_WS2812B-2020_PLCC4_2.0x2.0mm - no silkscreen"
 			(at 210.185 96.52 0)
 			(hide yes)
@@
 			)
 		)
-		(property "Footprint" "footprints:LED_WS2812B-2020_PLCC4_2.0x2.0mm - no silkscreen"
+		(property "Footprint" "easyeda2kicad:LED_WS2812B-2020_PLCC4_2.0x2.0mm - no silkscreen"
 			(at 231.14 96.52 0)
 			(hide yes)
@@
 			)
 		)
-		(property "Footprint" "footprints:LED_WS2812B-2020_PLCC4_2.0x2.0mm - no silkscreen"
+		(property "Footprint" "easyeda2kicad:LED_WS2812B-2020_PLCC4_2.0x2.0mm - no silkscreen"
 			(at 168.275 96.52 0)
 			(hide yes)

Commit message: old 2020 discontinued.. switch to new one
Parts:
- D1, D10, D11, D12, D13, D14, D15, D16, D17, D18, D19, D2, D20, D21, D22, D23, D24, D3, D4, D5, D6, D7, D8, D9: LCSC Part # C965555 -> C52917434
