File: hardware/triangle/usb_and_power.kicad_sch (KiCad schematic)
At the start: 18 parts, among them J1 USB_C_Receptacle_USB2.0_16P, J2 USB_C_Receptacle_USB2.0_16P, U2 EA8212HT6R

Commit message: triangle tiles v3
Parts:
- removed D25, D26: ESD8351XV2T1G_C19829478, easyeda2kicad:SOD-523_L1.2-W0.8-LS1.6-RD, symbol easyeda2kicad:ESD8351XV2T1G_C19829478
- removed D27, D28: SMAJ15A_C19077535, easyeda2kicad:SMA_L4.3-W2.6-LS5.0-RD, symbol easyeda2kicad:SMAJ15A_C19077535
Other:
- moved on the sheet: C34, J2
