File: hardware/input/input.kicad_pcb (KiCad board)
At the start: 2 copper layers, 80 x 60 mm, 18 parts, among them SW1 EVP-ASAC1A, SW2 EVP-ASAC1A, SW3 EVP-ASAC1A, SW4 EVP-ASAC1A, SW5 EVP-ASAC1A, SW6 CL-SB-13A-02T, U1 MCP23008T-E/SS

Commit message: more input board work
Parts:
- moved C1 14.8 mm to (172.8, 125.0), turned to -90 degrees
- moved C2 14.0 mm to (171.2, 125.5)
- moved R1 11.8 mm to (169.2, 125.5), turned to -90 degrees
- moved C3 4.51 mm to (143.8, 89.5), turned to 180 degrees
- moved C4 4.28 mm to (143.5, 119.5), turned to -90 degrees
- moved SW1 3.00 mm to (131.0, 91.0)
- moved SW2 3.00 mm to (131.0, 129.0)
- moved SW3 3.00 mm to (112.0, 110.0)
- moved SW4 3.00 mm to (150.0, 110.0)
- moved SW5 3.00 mm to (131.0, 110.0)
Routing:
- net BTN LEFT: track 0.00 -> 58.6 mm, vias 0 -> 1
- net IR SENSOR DATA: track 0.00 -> 56.1 mm, vias 0 -> 1
- net GND: track 0.00 -> 47.0 mm, vias 0 -> 17
- net BTN DOWN: track 0.00 -> 44.2 mm, vias 0 -> 1
- net SOUND REACTIVE OFF: track 0.00 -> 38.6 mm, vias 0 -> 1
- net BTN CENTER: track 0.00 -> 35.2 mm, vias 0 -> 1
- net SOUND REACTIVE ON: track 0.00 -> 33.9 mm, vias 0 -> 1
- net BTN UP: track 0.00 -> 30.4 mm, vias 0 -> 1
- net +3.3V: track 0.00 -> 19.0 mm, vias 0 -> 9
- net BTN RIGHT: track 0.00 -> 7.32 mm, vias 0 -> 1
- net Net-(CGQ1-VCC): track 0.00 -> 5.97 mm, vias 0 -> 1
- net USB-C D-: track 0.00 -> 3.94 mm
- net USB-C D+: track 0.00 -> 3.90 mm
- added copper zone on In2.Cu, net +3.3V
- added copper zone on In1.Cu, net GND
Other:
- copper layers 2 -> 4

Commit message: a few more changes for the input board
Parts:
- moved C4 19.9 mm to (134.0, 102.0), turned to 180 degrees
- moved U1 16.8 mm to (138.8, 98.2), turned to -90 degrees
- moved C1 9.72 mm to (163.5, 122.0), turned to 90 degrees
- moved C2 7.42 mm to (165.0, 121.5), turned to -90 degrees
- moved R1 4.59 mm to (167.0, 121.5), turned to 90 degrees
- moved C3 0.75 mm to (144.0, 90.2)
Connections:
- U1 pad 12: BTN UP -> SOUND REACTIVE OFF
- U1 pad 13: BTN DOWN -> SOUND REACTIVE ON
- U1 pad 14: BTN LEFT -> BTN RIGHT
- U1 pad 15: BTN RIGHT -> BTN DOWN
- U1 pad 17: SOUND REACTIVE ON -> BTN LEFT
- U1 pad 18: SOUND REACTIVE OFF -> BTN UP
Routing:
- net BTN LEFT: track 58.6 -> 35.4 mm
- net BTN UP: track 30.4 -> 15.0 mm
- net BTN CENTER: track 35.2 -> 22.0 mm
- net USB-C CC1&CC2: track 0.00 -> 12.6 mm, vias 0 -> 3
- net BTN DOWN: track 44.2 -> 31.7 mm
- net SOUND REACTIVE ON: track 33.9 -> 26.0 mm
- net SOUND REACTIVE OFF: track 38.6 -> 30.8 mm
- net USB-C D-: track 3.94 -> 11.7 mm
- net USB-C D+: track 3.90 -> 10.4 mm
- net GND: track 47.0 -> 52.1 mm, vias 17 -> 19
- net BTN RIGHT: track 7.32 -> 12.0 mm
- net +3.3V: track 19.0 -> 21.0 mm
